File: Matt3o/Matt3o-CA.kicad_pcb (KiCad board)
At the start: 2 copper layers, 284.5 x 94 mm, 219 parts, among them IC1 ATMEGA32U4, K1 AVR_ICSP, P1 CONN_4, P2 CONN_4, SW1 TILDE, SW10 FN, SW11 2, SW12 W, SW13 S, SW14 X, SW15 ALT, SW16 3, SW17 E, SW18 D, SW19 C, SW2 TAB, SW20 4, SW21 R, SW22 F, SW23 V, SW24 5, SW25 T, SW26 G, SW27 B, SW28 SPACE, SW29 6, SW3 CAPS, SW30 Y, SW31 H, SW32 N, SW33 7, SW34 U, SW35 J, SW36 M, SW37 8, SW38 I, SW39 K, SW4 SHIFT, SW40 ,, SW41 9, SW42 O, SW43 L, SW44 ., SW45 ALT_R, SW46 0, SW47 P, SW48 ;, SW49 /, SW5 CTRL, SW50 CTRL_R, SW51 -, SW52 {, SW53 ', SW54 SHIFT_R, SW55 LEFT, SW56 =, SW57 }, SW58 ENTER, SW59 BCKSP, SW6 1, SW60 |, SW61 UP, SW62 DOWN, SW63 INS, SW64 DEL, SW65 PRINT, SW66 PAUSE, SW67 RIGHT, SW7 Q, SW8 A, SW9 Z, X1 ASX4

Commit message: cut layer. 286,5 x 96,5 mm.
Routing:
- net /SCK: track 5.97 -> 4.78 mm
- net /ROW1: track 421.4 -> 422.6 mm
Other:
- board size 284.5 x 94 mm -> 286.1 x 96.2 mm
- board text added: "GH65 Cherry-Alps design by Agodinhost"
Changed lines of the file:
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@@
     (area 150.791334 151.434801 449.453002 253.936501)
     (thickness 1.6002)
-    (drawings 6)
+    (drawings 7)
     (tracks 964)
     (zones 0)
@@
     (pad_drill 1.501139)
     (pad_to_mask_clearance 0.254)
-    (aux_axis_origin 0 0)
+    (aux_axis_origin 151.9428 157.5816)
     (visible_elements 7FFE7FBF)
     (pcbplotparams
@@
     )
   )
-  (dimension 94.996 (width 0.3048) (layer Cmts.User)
-    (gr_text "94,996 mm" (at 442.6966 205.867 90) (layer Cmts.User)
+  (gr_text "GH65 Cherry-Alps\ndesign by Agodinhost" (at 242.697 243.0526) (layer Dwgs.User)
+    (effects (font (size 2.032 1.524) (thickness 0.3048)))
+  )
+  (dimension 286.512001 (width 0.3048) (layer Cmts.User)
+    (gr_text "286,512 mm" (at 295.199396 150.863299 359.9949206) (layer Cmts.User)
       (effects (font (size 2.032 1.524) (thickness 0.3048)))
     )
-    (feature1 (pts (xy 438.023 158.369) (xy 444.3222 158.369)))
-    (feature2 (pts (xy 438.023 253.365) (xy 444.3222 253.365)))
-    (crossbar (pts (xy 441.071 253.365) (xy 441.071 158.369)))
-    (arrow1a (pts (xy 441.071 158.369) (xy 441.65742 159.495503)))
-    (arrow1b (pts (xy 441.071 158.369) (xy 440.48458 159.495503)))
-    (arrow2a (pts (xy 441.071 253.365) (xy 441.65742 252.238497)))
-    (arrow2b (pts (xy 441.071 253.365) (xy 440.48458 252.238497)))
+    (feature1 (pts (xy 438.4548 157.607) (xy 438.45554 149.2504)))
+    (feature2 (pts (xy 151.9428 157.5816) (xy 151.94354 149.225)))
+    (crossbar (pts (xy 151.943252 152.476199) (xy 438.455252 152.501599)))
+    (arrow1a (pts (xy 438.455252 152.501599) (xy 437.328697 153.087919)))
+    (arrow1b (pts (xy 438.455252 152.501599) (xy 437.328801 151.915079)))
+    (arrow2a (pts (xy 151.943252 152.476199) (xy 153.069703 153.062719)))
+    (arrow2b (pts (xy 151.943252 152.476199) (xy 153.069807 151.889879)))
   )
-  (dimension 285.369 (width 0.3048) (layer Cmts.User)
-    (gr_text "285,369 mm" (at 295.2115 153.314401) (layer Cmts.User)
+  (dimension 96.596203 (width 0.3048) (layer Cmts.User)
+    (gr_text "96,596 mm" (at 442.226698 205.904113 270.0150659) (layer Cmts.User)
       (effects (font (size 2.032 1.524) (thickness 0.3048)))
     )
-    (feature1 (pts (xy 152.527 158.369) (xy 152.527 151.688801)))
-    (feature2 (pts (xy 437.896 158.369) (xy 437.896 151.688801)))
-    (crossbar (pts (xy 437.896 154.940001) (xy 152.527 154.940001)))
-    (arrow1a (pts (xy 152.527 154.940001) (xy 153.653503 154.353581)))
-    (arrow1b (pts (xy 152.527 154.940001) (xy 153.653503 155.526421)))
-    (arrow2a (pts (xy 437.896 154.940001) (xy 436.769497 154.353581)))
-    (arrow2b (pts (xy 437.896 154.940001) (xy 436.769497 155.526421)))
-  )
-  (gr_line (start 437.5658 252.8697) (end 153.0858 252.8697) (angle 90) (layer Edge.Cuts) (width 0.381))
-  (gr_line (start 437.56834 158.8897) (end 437.56834 252.8697) (angle 90) (layer Edge.Cuts) (width 0.381))
-  (gr_line (start 153.0858 252.8697) (end 153.0858 158.8897) (angle 90) (layer Edge.Cuts) (width 0.381))
-  (gr_line (start 153.0858 158.8897) (end 437.5658 158.8897) (angle 90) (layer Edge.Cuts) (width 0.381))
+    (feature1 (pts (xy 438.4802 254.2032) (xy 443.864998 254.201786)))
+    (feature2 (pts (xy 438.4548 157.607) (xy 443.839598 157.605586)))
+    (crossbar (pts (xy 440.588399 157.60644) (xy 440.613799 254.20264)))
+    (arrow1a (pts (xy 440.613799 254.20264) (xy 440.027083 253.076291)))
+    (arrow1b (pts (xy 440.613799 254.20264) (xy 441.199923 253.075983)))
+    (arrow2a (pts (xy 440.588399 157.60644) (xy 440.002275 158.733097)))
+    (arrow2b (pts (xy 440.588399 157.60644) (xy 441.175115 158.732789)))
+  )
+  (gr_line (start 152.146 157.7848) (end 152.146 254) (angle 90) (layer Edge.Cuts) (width 0.381))
+  (gr_line (start 438.2516 157.8102) (end 152.146 157.7848) (angle 90) (layer Edge.Cuts) (width 0.381))
+  (gr_line (start 438.2516 157.8102) (end 438.277 254) (angle 90) (layer Edge.Cuts) (width 0.381))
+  (gr_line (start 152.1714 254) (end 438.2262 254) (angle 90) (layer Edge.Cuts) (width 0.381))
   (segment (start 295.1353 239.0902) (end 295.148 239.0775) (width 0.4064) (layer Back) (net 0))
   (segment (start 175.9966 235.712) (end 176.022 235.6866) (width 0.4064) (layer Front) (net 0))
@@
   (segment (start 303.2633 234.1626) (end 303.2633 233.8705) (width 0.4064) (layer Back) (net 23))
   (segment (start 324.993 234.8992) (end 321.7672 231.6734) (width 0.4064) (layer Back) (net 23))
+  (segment (start 324.993 236.093) (end 324.993 234.8992) (width 0.4064) (layer Back) (net 23))
   (segment (start 317.9318 222.0468) (end 313.6519 217.7669) (width 0.4064) (layer Back) (net 24))
   (segment (start 310.3753 217.7669) (end 310.3753 217.7429) (width 0.4064) (layer Back) (net 24))
@@
   (segment (start 310.6928 235.4326) (end 321.9958 235.4326) (width 0.4064) (layer Back) (net 27))
   (segment (start 307.848 238.2774) (end 310.6928 235.4326) (width 0.4064) (layer Back) (net 27))
-  (segment (start 324.993 236.093) (end 324.993 234.8992) (width 0.4064) (layer Back) (net 28))
   (segment (start 324.993 239.27054) (end 324.993 236.093) (width 0.4064) (layer Back) (net 28))
   (segment (start 303.2633 235.7628) (end 303.2633 234.1626) (width 0.4064) (layer Back) (net 28))
@@
     (polygon
       (pts
-        (xy 437.9976 158.369) (xy 152.4254 158.3436) (xy 152.4254 253.4158) (xy 437.9976 253.4158) (xy 437.9976 158.369)
+        (xy 437.388 253.238) (xy 152.908 253.238) (xy 152.908 158.75) (xy 437.388 158.75)
       )
     )
@@
     (polygon
       (pts
-        (xy 437.9976 158.369) (xy 152.4254 158.3436) (xy 152.4254 253.4158) (xy 437.9976 253.4158) (xy 437.9976 158.369)
+        (xy 437.388 253.238) (xy 152.908 253.238) (xy 152.908 158.75) (xy 437.388 158.75)
       )
     )

Commit message: review moving diodes out of switch area.
Parts:
- moved D45 3.62 mm to (344.9, 235.7), turned to 180 degrees
- moved D67 3.32 mm to (425.9, 235.7)
- moved D62 3.26 mm to (406.8, 235.7)
- moved D55 2.62 mm to (385.3, 235.7)
- moved D58 2.60 mm to (397.6, 197.6)
- moved D50 2.58 mm to (364.0, 235.7)
- moved D10 2.57 mm to (182.9, 235.7)
- moved D5 2.51 mm to (161.4, 235.7)
Connections:
- IC1 pad 9: /SCK -> /ROW1
- K1 pad 3: /SCK -> /ROW1
- SW12 pad 1: /ROW3 -> /MISO
- SW13 pad 1: /ROW2 -> /MOSI
- SW17 pad 1: /ROW3 -> /MISO
- SW18 pad 1: /ROW2 -> /MOSI
- SW2 pad 1: /ROW3 -> /MISO
- SW21 pad 1: /ROW3 -> /MISO
- SW22 pad 1: /ROW2 -> /MOSI
- SW25 pad 1: /ROW3 -> /MISO
- SW26 pad 1: /ROW2 -> /MOSI
- SW3 pad 1: /ROW2 -> /MOSI
- SW30 pad 1: /ROW3 -> /MISO
- SW31 pad 1: /ROW2 -> /MOSI
- SW34 pad 1: /ROW3 -> /MISO
- SW35 pad 1: /ROW2 -> /MOSI
- SW38 pad 1: /ROW3 -> /MISO
- SW39 pad 1: /ROW2 -> /MOSI
- SW42 pad 1: /ROW3 -> /MISO
- SW43 pad 1: /ROW2 -> /MOSI
- SW47 pad 1: /ROW3 -> /MISO
- SW48 pad 1: /ROW2 -> /MOSI
- SW52 pad 1: /ROW3 -> /MISO
- SW53 pad 1: /ROW2 -> /MOSI
- SW57 pad 1: /ROW3 -> /MISO
- SW58 pad 1: /ROW2 -> /MOSI
- SW60 pad 1: /ROW3 -> /MISO
- SW64 pad 1: /ROW3 -> /MISO
- SW65 pad 1: /ROW2 -> /MOSI
- SW7 pad 1: /ROW3 -> /MISO
- SW8 pad 1: /ROW2 -> /MOSI
Routing:
- net /ROW3: track 453.0 -> 0.00 mm
- net /MISO: track 45.0 -> 498.1 mm
- net /ROW2: track 419.5 -> 0.00 mm
- net /MOSI: track 45.3 -> 464.7 mm
- net /ROW1: track 422.6 -> 427.4 mm
- net /SCK: track 4.78 -> 0.00 mm
- net N-0000075: track 10.3 -> 14.7 mm
- net N-0000015: track 10.3 -> 13.7 mm
- net N-000005: track 10.3 -> 13.7 mm
- net N-000008: track 10.3 -> 13.1 mm
- net N-0000071: track 10.3 -> 13.0 mm
- net /COL9: track 124.2 -> 121.6 mm
- net N-000003: track 10.3 -> 12.9 mm
- net /COL10: track 141.3 -> 138.7 mm
- net /COL11: track 165.6 -> 163.0 mm
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
Commit message: final version touches.
Parts:
- added HOLE: VAL**, hole-round, F.Cu at (171.4, 177.3)
- added HOLE: VAL**, hole-round, F.Cu at (400.0, 177.3)
- added HOLE: VAL**, hole-round, F.Cu at (419.0, 234.5)
- added HOLE: VAL**, hole-round, F.Cu at (195.2, 234.5)
- added HOLE: VAL**, hole-round, F.Cu at (252.4, 196.4)
- added HOLE: VAL**, hole-round, F.Cu at (338.1, 215.4)
- moved D25 16.7 mm to (252.4, 178.6)
- moved C7 13.1 mm to (285.7, 177.3), turned to 90 degrees
- moved C6 10.9 mm to (283.3, 177.3), turned to 90 degrees
- moved C5 9.38 mm to (280.9, 177.3), turned to 90 degrees
- moved C4 8.89 mm to (278.4, 177.3), turned to 90 degrees
- moved D28 5.04 mm to (267.1, 240.5), turned to 90 degrees
- moved D43 3.44 mm to (332.0, 214.2)
- moved D9 3.40 mm to (189.1, 233.2)
- moved R2 3.33 mm to (290.1, 209.7)
- moved D19 2.60 mm to (228.6, 216.7)
- moved D23 2.60 mm to (247.7, 216.7)
- moved D32 2.60 mm to (285.8, 216.7)
- moved D36 2.60 mm to (304.8, 216.7)
- moved D40 2.60 mm to (323.9, 216.7)
- moved D15 2.54 mm to (204.3, 235.7)
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Routing:
- net /MOSI: track 464.7 -> 488.9 mm
- net GND: track 59.2 -> 49.2 mm
- net /SCL: track 55.7 -> 46.9 mm
- net /COL5: track 118.0 -> 125.2 mm
- net /COL4: track 131.5 -> 137.6 mm
- net /D+: track 52.7 -> 47.7 mm
- net /COL6: track 88.8 -> 93.5 mm
- net /D-: track 48.3 -> 52.9 mm
- net /COL1: track 210.9 -> 206.4 mm
- net /COL8: track 122.9 -> 126.3 mm
- net /MISO: track 498.1 -> 501.2 mm
- net N-0000066: track 10.3 -> 13.5 mm
- net /COL7: track 79.2 -> 82.2 mm
- net N-0000096: track 10.3 -> 12.9 mm
- net N-0000081: track 10.3 -> 12.9 mm
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