File: GH-MXAlps-mini/GH-MXAlps-mini.kicad_pcb (KiCad board)
At the start: 2 copper layers, 182 parts, among them IC1 ATMEGA32U4, K1 AVR_ICSP, P1 CONN_4, P2 CONN_4, SW1 K_ESC, SW10 K_A, SW11 K_Z, SW12 K_ALT, SW13 K_F2, SW14 K_2, SW15 K_W, SW16 K_S, SW17 K_X, SW18 K_SPACE, SW19 K_F3, SW2 K_` ~, SW20 K_3, SW21 K_E, SW22 K_D, SW23 K_C, SW24 K_F4, SW25 K_4, SW26 K_R, SW27 K_F, SW28 K_V, SW29 K_F5, SW3 K_TAB, SW30 K_5, SW31 K_T, SW32 K_G, SW33 K_B, SW34 K_F6, SW35 K_6, SW36 K_Y, SW37 K_H, SW38 K_N, SW39 K_F7, SW4 K_CAPS, SW40 K_7, SW41 K_U, SW42 K_J, SW43 K_M, SW44 K_F8, SW45 K_8, SW46 K_I, SW47 K_K, SW48 K_< ,, SW49 K_F9, SW5 K_SHIFT, SW50 K_9, SW51 K_O, SW52 K_L, SW53 K_> ., SW54 K_ALT_R, SW55 K_F10, SW56 K_0, SW57 K_P, SW58 K_; :, SW59 K_/ ?, SW6 K_CTRL, SW60 K_CTRL_R, SW61 K_F11, SW62 K_- _, SW63 K_[ {, SW64 K_' ", SW65 K_SHIFT_R, SW66 K_LEFT, SW67 K_F12, SW68 K_= +, SW69 K_] }, SW7 K_F1, SW70 K_ENTER, SW71 K_UP, SW72 K_DOWN, SW73 K_PrtSc, SW74 K_Pause, SW75 K_Backspace, SW76 K_\ |, SW77 K_Delete, SW78 K_Home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

Commit message: 1U = 1.90mm
Parts:
- moved P2 175.2 mm to (194.8, 218.5), turned to 90 degrees
- moved P1 169.5 mm to (199.5, 218.5), turned to 90 degrees
- moved IC1 167.9 mm to (166.2, 218.5)
- moved C1 164.0 mm to (190.6, 223.4)
- moved C2 164.0 mm to (190.6, 218.7)
- moved C3 164.0 mm to (190.6, 213.9)
- moved C4 164.0 mm to (185.8, 223.4)
- moved C5 164.0 mm to (181.1, 218.7)
- moved C6 164.0 mm to (181.1, 223.4)
- moved C7 164.0 mm to (181.1, 213.9)
- moved R1 164.0 mm to (185.8, 218.7)
- moved R2 164.0 mm to (176.3, 213.9)
- moved R3 164.0 mm to (176.3, 223.4)
- moved R4 164.0 mm to (185.8, 213.9)
- moved R5 164.0 mm to (176.3, 218.7)
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Other:
- board text added: "1u = 19,00mm 1/2 u = 9,50mm 1/4 u = 4,75mm"
- board text removed: "1u = 19,05mm 1/2 u = 9,525mm 1/4 u = 4,7625mm"
